File: Control/Control_PCB/Control_PCB.kicad_sch (KiCad schematic)
At the start: 119 parts, among them J1 Motor_cont2, J10 NC, J11 IOREF, J12 RESET, J13 +3V3, J14 +5V_1, J15 GND1, J16 GND2, J17 VIN, J18 AD0, J19 AD1, J2 Motor_cont1, J20 AD2, J21 AD3, J22 AD4, J23 AD5, J24 AD6, J25 AD7, J26 AD8, J27 AD9, J28 AD10, J29 AD11, J3 Driver1, J30 AD12, J31 AD13, J32 AD14, J33 AD15, J34 +5V_3, J35 23, J36 25, J37 27, J38 29, J39 31, J4 ARM, J40 33, J41 35, J42 37, J43 39, J44 41, J45 43, J46 45, J47 47, J48 49, J49 51, J5 Encoder2, J50 53, J51 GND5, J52 SCL, J53 SDA, J54 AREF, J55 GND3, J56 13, J57 12, J58 11, J59 10, J6 Encoder1, J60 9, J61 8, J62 7, J63 6, J64 5, J65 4, J66 3, J67 2, J68 1, J69 0, J7 Router_Power, J70 21, J71 20, J72 19, J73 18, J74 17, J75 16, J76 15, J77 14, J78 +5V_2, J79 22, J8 Metal_Sensor, J80 24, J81 26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

Commit message: Second commit
Parts:
- added J98: to_power, Connector_JST:JST_XH_B10B-XH-A_1x10_P2.50mm_Vertical, symbol Connector:Screw_Terminal_01x10
- C1, C2, C3: value 20p -> 220n; footprint Capacitor_THT:C_Disc_D5.0mm_W2.5mm_P5.00mm -> Capacitor_THT:C_Disc_D7.5mm_W5.0mm_P7.50mm
- J1, J2, J3, J97: footprint TerminalBlock_TE-Connectivity:TerminalBlock_TE_282834-3_1x03_P2.54mm_Horizontal -> Connector_JST:JST_XH_B3B-XH-A_1x03_P2.50mm_Vertical
- J4: footprint TerminalBlock_TE-Connectivity:TerminalBlock_TE_282834-8_1x08_P2.54mm_Horizontal -> Connector_JST:JST_XH_B8B-XH-A_1x08_P2.50mm_Vertical
- J5, J6: footprint TerminalBlock_TE-Connectivity:TerminalBlock_TE_282834-6_1x06_P2.54mm_Horizontal -> Connector_JST:JST_XH_B6B-XH-A_1x06_P2.50mm_Vertical
- J7, J9: footprint TerminalBlock_TE-Connectivity:TerminalBlock_TE_282834-2_1x02_P2.54mm_Horizontal -> MyLibrary:TerminalBlock_bornier-2_P5.08mm
- J8: footprint TerminalBlock_TE-Connectivity:TerminalBlock_TE_282834-3_1x03_P2.54mm_Horizontal -> MyLibrary:TerminalBlock_bornier-3_P5.08mm
- J96: footprint TerminalBlock_TE-Connectivity:TerminalBlock_TE_282834-2_1x02_P2.54mm_Horizontal -> Connector_JST:JST_XH_B2B-XH-A_1x02_P2.50mm_Vertical
- Q1, Q2: footprint Package_TO_SOT_THT:TO-92_Inline -> Package_TO_SOT_THT:TO-92L_Inline_Wide
- R1: value 100k -> 1M
- R2: value 12M -> 1M
- R3: value 12M -> 330K
- U6, U8: footprint External_footprint_lib:MODULE_ZC576300 -> MyLibrary:MODULE_ZC576300
Connections:
- net res_t is gone; now on net battery_vcc: R1.1, U9.4 (R)
- net DAC1_Out: now also J2.2 (Pin_2); no longer J2.3 (Pin_3)
- net DAC2_Out: now also J2.3 (Pin_3); no longer J2.2 (Pin_2)
- net GND: now also J98.10 (Pin_10)
- net LIS: now also A1.12, J57.1 (Pin_1)
- net RIS: now also A1.13, J56.1 (Pin_1)
- net battery_gnd: now also U10.10 (R), U10.4 (R), U10.6 (S), U10.8 (S), U11.10 (R), U11.4 (R), U11.6 (S), U11.8 (S), U5.12, U5.13
- net 17: now reaches A1.17, J74.1 (Pin_1)
- net 17: now also J98.6 (Pin_6)
- net 1: now reaches A1.1, J68.1 (Pin_1)
- net 1: now also J98.5 (Pin_5)
- net 0: now reaches A1.0, J69.1 (Pin_1)
- net 0: now also J98.8 (Pin_8)
- net 10: now reaches A1.10, J59.1 (Pin_1)
- net 10: now also J98.2 (Pin_2)
- net 11: now reaches A1.11, J58.1 (Pin_1)
- net 11: now also J98.1 (Pin_1)
- net 9: now reaches A1.9, J60.1 (Pin_1)
- net 9: now also J98.3 (Pin_3)
- net 8: now reaches A1.8, J61.1 (Pin_1)
- net 8: now also J98.4 (Pin_4)
- net 14: now reaches A1.14, J77.1 (Pin_1)
- net 15: now reaches A1.15, J76.1 (Pin_1)
- net 15: now also J98.9 (Pin_9)
- net 16: now reaches A1.16, J75.1 (Pin_1)
- net 16: now also J98.7 (Pin_7)
- no-connect marks 18 -> 6

Commit message: Third commit
Parts:
- added J100, J101: MPU1, MyLibrary:module_mpu6050, symbol Connector:Screw_Terminal_01x08
- added J99: TTL, Connector_JST:JST_XH_B4B-XH-A_1x04_P2.50mm_Vertical, symbol Connector:Screw_Terminal_01x04
Connections:
- net GND: now also J100.2 (Pin_2), J101.2 (Pin_2), J99.4 (Pin_4)
- net SCL: now also J100.3 (Pin_3), J101.3 (Pin_3)
- net SDA: now also J100.4 (Pin_4), J101.4 (Pin_4)
- net arduino_5V_out: now also J100.1 (Pin_1), J101.1 (Pin_1), J99.3 (Pin_3)
- net 23: now reaches A1.23, J35.1 (Pin_1)
- net 23: now also J98.9 (Pin_9)
- net 14 renamed TTL_RX
- net TTL_RX: now also J99.1 (Pin_1)
- net 15 renamed TTL_TX
- net TTL_TX: now also J99.2 (Pin_2); no longer J98.9 (Pin_9)
- no-connect marks 6 -> 14

Commit message: sixth commit
Connections:
- net 0: no longer J98.8 (Pin_8)
- net 1: no longer J98.5 (Pin_5)
- net 25: now reaches A1.25, J36.1 (Pin_1)
- net 25: now also J98.8 (Pin_8)
- net 27: now reaches A1.27, J37.1 (Pin_1)
- net 27: now also J98.5 (Pin_5)
Changed lines of the file:
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@@
+		)
+	)
+	(label "25"
+		(at 201.93 176.53 270)
+		(fields_autoplaced yes)
+		(effects
+			(font
+				(size 1.27 1.27)
+			)
+			(justify right bottom)
 		)
 	)
@@
 		)
 	)
+	(label "27"
+		(at 194.31 176.53 270)
+		(fields_autoplaced yes)
+		(effects
+			(font
+				(size 1.27 1.27)
+			)
+			(justify right bottom)
+		)
+	)
 	(label "battery_gnd"
 		(at 115.57 86.36 180)
@@
 		)
 	)
+	(label "25"
+		(at 210.82 123.19 180)
+		(fields_autoplaced yes)
+		(effects
+			(font
+				(size 1.27 1.27)
+			)
+			(justify right bottom)
+		)
+	)
 	(label "SCL"
 		(at 269.24 179.07 270)
@@
 		)
 	)
-	(label "1"
-		(at 194.31 176.53 270)
-		(fields_autoplaced yes)
-		(effects
-			(font
-				(size 1.27 1.27)
-			)
-			(justify right bottom)
-		)
-	)
 	(label "battery_gnd"
 		(at 266.7 26.67 270)
@@
 		)
 	)
-	(label "0"
-		(at 201.93 176.53 270)
-		(fields_autoplaced yes)
-		(effects
-			(font
-				(size 1.27 1.27)
-			)
-			(justify right bottom)
-		)
-	)
 	(label "LEN"
 		(at 251.46 80.01 0)
@@
 		)
 	)
+	(label "27"
+		(at 210.82 125.73 180)
+		(fields_autoplaced yes)
+		(effects
+			(font
+				(size 1.27 1.27)
+			)
+			(justify right bottom)
+		)
+	)
